File: KiCAD design/KiCAD design.kicad_sch (KiCad schematic)
At the start: 1 part, among them U101 NUCLEO64-F411RE

Commit message: add link to switch and 1k resistor
Parts:
- U101: Price (none) -> x; PurchaseLoc (none) -> x
Changed lines of the file:
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@@
+      (effects (font (size 1.27 1.27)) hide)
+    )
+    (property "Price" "x" (id 4) (at 93.98 149.86 0)
+      (effects (font (size 1.27 1.27)) hide)
+    )
+    (property "PurchaseLoc" "x" (id 5) (at 93.98 149.86 0)
       (effects (font (size 1.27 1.27)) hide)
     )
