File: KiCAD design/on_board_components.kicad_sch (KiCad schematic)
At the start: 11 parts, among them U401 ACS712xLCTR-20A

Commit message: change voltage dividor resistors to larger dimensions
Parts:
- R404: PurchaseLoc https://www.digikey.fi/en/products/detail/yageo/AC0402FR-07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 -> https://www.digikey.fi/en/products/detail/yageo/RC0805JR-07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
- R405: PurchaseLoc https://www.digikey.fi/en/products/detail/yageo/AC0402FR-07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 -> https://www.digikey.fi/en/products/detail/yageo/RC0805FR-07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
Changed lines of the file:
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@@
       (effects (font (size 1.27 1.27)) hide)
     )
-    (property "PurchaseLoc" "https://www.digikey.fi/en/products/detail/yageo/AC0402FR-0710KL/5895030" (id 4) (at 81.28 60.96 0)
+    (property "PurchaseLoc" "https://www.digikey.fi/en/products/detail/yageo/RC0805JR-0710KL/728241" (id 4) (at 81.28 60.96 0)
       (effects (font (size 1.27 1.27)) hide)
     )
@@
       (effects (font (size 1.27 1.27)) hide)
     )
-    (property "PurchaseLoc" "https://www.digikey.fi/en/products/detail/yageo/AC0402FR-0719K1L/5895123" (id 4) (at 81.28 71.12 0)
-      (effects (font (size 1.27 1.27)) hide)
-    )
+    (property "PurchaseLoc" "https://www.digikey.fi/en/products/detail/yageo/RC0805FR-0719K1L/727656" (id 4) (at 81.28 71.12 0)
+      (effects (font (size 1.27 1.27)) hide)
+    )

Commit message: more comments (no changes in functionality)
Other:
- note added: "Current sensor for measuring the power draw of the robot."
- note added: "Current sensor output is 0..5 V, Nucleo ADC pin input is 0..3.3 V. Voltage divider is required."
- note added: "Operational and error LEDs."
- note removed: "Current sensor output is 0..5 V, Nucleo ADC pin input is 0..3.3 V. Needs voltage divider"
Changed lines of the file:
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@@
     (effects (font (size 3.81 3.81)) (justify left bottom))
   )
-  (text "Current sensor output is 0..5 V,\nNucleo ADC pin input is 0..3.3 V.\nNeeds voltage divider"
+  (text "Current sensor output is 0..5 V,\nNucleo ADC pin input is 0..3.3 V.\nVoltage divider is required."
     (at 77.47 55.88 0)
     (effects (font (size 1.27 1.27)) (justify left bottom))
@@
     (effects (font (size 3.81 3.81)) (justify left bottom))
   )
+  (text "Operational and error LEDs." (at 134.62 81.28 0)
+    (effects (font (size 1.27 1.27)) (justify left bottom))
+  )
+  (text "Current sensor for measuring the power draw of the robot."
+    (at 13.97 83.82 0)
+    (effects (font (size 1.27 1.27)) (justify left bottom))
+  )
   (hierarchical_label "IP+" (shape passive) (at 44.45 52.07 180)
