File: KiCAD design/ext_components.kicad_sch (KiCad schematic)
At the start: 5 parts

Commit message: end PCB
Parts:
- LiPo_bat401: Price 12.31 -> 13.42; PurchaseLoc https://hobbyking.com/en_us/turnigy-2200mah-3s-25c-lipo-pac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 -> https://hobbyking.com/en_us/zippy-compact-1800mah-3s-25c-li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
- TOF1, TOF2: Price 13.75 -> 12.07; PurchaseLoc https://www.digikey.fi/en/products/detail/adafruit-industri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 -> https://www.digikey.fi/en/products/detail/dfrobot/SEN0245/8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
Changed lines of the file:
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@@
       (effects (font (size 1.27 1.27)) hide)
     )
-    (property "PurchaseLoc" "https://hobbyking.com/en_us/turnigy-2200mah-3s-25c-lipo-pack.html" (id 4) (at 203.2 97.79 90)
+    (property "PurchaseLoc" "https://hobbyking.com/en_us/zippy-compact-1800mah-3s-25c-lipo-pack.html" (id 4) (at 203.2 97.79 90)
       (effects (font (size 1.27 1.27)) hide)
     )
-    (property "Price" "12.31" (id 5) (at 203.2 97.79 90)
+    (property "Price" "13.42" (id 5) (at 203.2 97.79 90)
       (effects (font (size 1.27 1.27)) hide)
     )
@@
       (effects (font (size 1.27 1.27)) hide)
     )
-    (property "Datasheet" "https://cdn-learn.adafruit.com/downloads/pdf/adafruit-vl53l0x-micro-lidar-distance-sensor-breakout.pdf" (id 3) (at 94.742 140.97 0)
+    (property "Datasheet" "~" (id 3) (at 94.742 140.97 0)
       (effects (font (size 1.27 1.27)) hide)
     )
-    (property "PurchaseLoc" "https://www.digikey.fi/en/products/detail/adafruit-industries-llc/3317/6569762" (id 4) (at 93.98 135.89 0)
+    (property "PurchaseLoc" "https://www.digikey.fi/en/products/detail/dfrobot/SEN0245/8827827?s=N4IgTCBcDaIG4BsCsBmBAGAHiAugXyA" (id 4) (at 93.98 135.89 0)
       (effects (font (size 1.27 1.27)) hide)
     )
-    (property "Price" "13.75" (id 5) (at 93.98 135.89 0)
+    (property "Price" "12.07" (id 5) (at 93.98 135.89 0)
       (effects (font (size 1.27 1.27)) hide)
     )
@@
       (effects (font (size 1.27 1.27)) hide)
     )
-    (property "Datasheet" "https://cdn-learn.adafruit.com/downloads/pdf/adafruit-vl53l0x-micro-lidar-distance-sensor-breakout.pdf" (id 3) (at 112.522 140.97 0)
+    (property "Datasheet" "~" (id 3) (at 112.522 140.97 0)
       (effects (font (size 1.27 1.27)) hide)
     )
-    (property "PurchaseLoc" "https://www.digikey.fi/en/products/detail/adafruit-industries-llc/3317/6569762" (id 4) (at 111.76 135.89 0)
+    (property "PurchaseLoc" "https://www.digikey.fi/en/products/detail/dfrobot/SEN0245/8827827?s=N4IgTCBcDaIG4BsCsBmBAGAHiAugXyA" (id 4) (at 111.76 135.89 0)
       (effects (font (size 1.27 1.27)) hide)
     )
-    (property "Price" "13.75" (id 5) (at 111.76 135.89 0)
+    (property "Price" "12.07" (id 5) (at 111.76 135.89 0)
       (effects (font (size 1.27 1.27)) hide)
     )

Commit message: update lipo battery to something in stock
Parts:
- LiPo_bat401: Price 13.42 -> 12.31; PurchaseLoc https://hobbyking.com/en_us/zippy-compact-1800mah-3s-25c-li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 -> https://hobbyking.com/en_us/turnigy-2200mah-3s-25c-lipo-pac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
Changed lines of the file:
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@@
       (effects (font (size 1.27 1.27)) hide)
     )
-    (property "PurchaseLoc" "https://hobbyking.com/en_us/zippy-compact-1800mah-3s-25c-lipo-pack.html" (id 4) (at 203.2 97.79 90)
+    (property "PurchaseLoc" "https://hobbyking.com/en_us/turnigy-2200mah-3s-25c-lipo-pack.html" (id 4) (at 203.2 97.79 90)
       (effects (font (size 1.27 1.27)) hide)
     )
-    (property "Price" "13.42" (id 5) (at 203.2 97.79 90)
+    (property "Price" "12.31" (id 5) (at 203.2 97.79 90)
       (effects (font (size 1.27 1.27)) hide)
     )

Commit message: change TOF sensor to one in stock (still VL53L0X, same pins)
Parts:
- TOF1, TOF2: Price 12.07 -> 13.75; PurchaseLoc https://www.digikey.fi/en/products/detail/dfrobot/SEN0245/8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 -> https://www.digikey.fi/en/products/detail/adafruit-industri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
Changed lines of the file:
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@@
       (effects (font (size 1.27 1.27)) hide)
     )
-    (property "PurchaseLoc" "https://www.digikey.fi/en/products/detail/dfrobot/SEN0245/8827827?s=N4IgTCBcDaIG4BsCsBmBAGAHiAugXyA" (id 4) (at 93.98 135.89 0)
+    (property "PurchaseLoc" "https://www.digikey.fi/en/products/detail/adafruit-industries-llc/3317/6569762" (id 4) (at 93.98 135.89 0)
       (effects (font (size 1.27 1.27)) hide)
     )
-    (property "Price" "12.07" (id 5) (at 93.98 135.89 0)
+    (property "Price" "13.75" (id 5) (at 93.98 135.89 0)
       (effects (font (size 1.27 1.27)) hide)
     )
@@
       (effects (font (size 1.27 1.27)) hide)
     )
-    (property "PurchaseLoc" "https://www.digikey.fi/en/products/detail/dfrobot/SEN0245/8827827?s=N4IgTCBcDaIG4BsCsBmBAGAHiAugXyA" (id 4) (at 111.76 135.89 0)
+    (property "PurchaseLoc" "https://www.digikey.fi/en/products/detail/adafruit-industries-llc/3317/6569762" (id 4) (at 111.76 135.89 0)
       (effects (font (size 1.27 1.27)) hide)
     )
-    (property "Price" "12.07" (id 5) (at 111.76 135.89 0)
+    (property "Price" "13.75" (id 5) (at 111.76 135.89 0)
       (effects (font (size 1.27 1.27)) hide)
     )
